Commit message: Adicion de modelos .obj con texturas

File: src/simulation/urdf/openbot_v1.urdf (robot description, URDF)
Before this commit: robot openbot_v1, 8 links, 7 joints
Links:
- link arm1_link_1: geometry collision mesh filename=meshes/collision/arm1_link_collision.stl scale=0.0001 0.0001 0.0001; visual mesh filename=meshes/visual/arm1_link_1.obj scale=0.001 0.001 0.001
- link arm2_link_1: geometry collision mesh filename=meshes/collision/arm2_link_collision.stl scale=0.0001 0.0001 0.0001; visual mesh filename=meshes/visual/arm2_link_1.obj scale=0.001 0.001 0.001
- link arm3_link_1: geometry collision mesh filename=meshes/collision/arm3_link_collision.stl scale=0.0001 0.0001 0.0001; visual mesh filename=meshes/visual/arm3_link_1.obj scale=0.001 0.001 0.001
- link arm4_link_1: geometry collision mesh filename=meshes/collision/arm4_link_collision.stl scale=0.0001 0.0001 0.0001; visual mesh filename=meshes/visual/arm4_link_1.obj scale=0.001 0.001 0.001
- link base_link: geometry collision mesh filename=meshes/collision/base_link_collision.stl scale=0.0001 0.0001 0.0001; visual mesh filename=meshes/visual/base_link.obj scale=0.001 0.001 0.001
- link clamp2_link_1: geometry collision mesh filename=meshes/collision/clamp2_link_collision.stl scale=0.0001 0.0001 0.0001; visual mesh filename=meshes/visual/clamp2_link_1.obj scale=0.001 0.001 0.001
- link clamp_arm_link_1: geometry collision mesh filename=meshes/collision/clamp_arm_link_collision.stl scale=0.0001 0.0001 0.0001; visual mesh filename=meshes/visual/clamp_arm_link_1.obj scale=0.001 0.001 0.001

Commit message: Cambios en rangos de movimiento del robot, adicion de coneccion con robot y seleccion de puerto serial

File: src/simulation/urdf/openbot_v1.urdf (robot description, URDF)
Before this commit: robot openbot_v1, 8 links, 7 joints
Joints:
- joint clamp1_clamp2_joint: limit lower=0.0 upper=1.57 effort=10 velocity=3 -> lower=-0.66 upper=1.57 effort=10 velocity=3

Commit message: Corrección de controlador de simulacion, adicion inicial de graficas

File: src/simulation/urdf/openbot_v1.urdf (robot description, URDF)
Before this commit: robot openbot_v1, 8 links, 7 joints
Joints:
- joint arm1_arm2_joint: limit lower=-1.6 upper=1.6 effort=10 velocity=3 -> lower=-2.617 upper=2.617 effort=10 velocity=3
- joint arm2_arm3_joint: limit lower=-2.09 upper=2.09 effort=10 velocity=3 -> lower=-2.617 upper=2.617 effort=10 velocity=3
- joint arm4_clamp1_joint: limit lower=-2.61 upper=1.57 effort=10 velocity=3 -> lower=-2.617 upper=2.617 effort=10 velocity=3
- joint clamp1_clamp2_joint: limit lower=-0.66 upper=1.57 effort=10 velocity=3 -> lower=-2.617 upper=2.617 effort=10 velocity=3

Commit message: Cambios al modelo 3D, giro de pinza y ajustes en la simulación

File: src/simulation/urdf/openbot_v1.urdf (robot description, URDF)
Before this commit: robot openbot_v1, 8 links, 7 joints
Joints:
- joint clamp1_clamp2_joint: origin xyz=0.018074 0.000709 0.070177 rpy=0 0 0 -> xyz=0.012074 0.028709 0.070177 rpy=0 0 1.5708
