Commit message: Algoritmo de pick and place

File: src/resources/pybullet/urdf/openbot_v1.urdf (robot description, URDF)
Before this commit: robot openbot_v1, 8 links, 7 joints
Links:
- link arm1_link_1: geometry collision mesh filename=meshes/collision/arm1_link_1_vhacd.obj scale=0.001 0.001 0.001; visual mesh filename=meshes/visual/arm1_link_1.obj scale=0.001 0.001 0.001
- link arm2_link_1: geometry collision mesh filename=meshes/collision/arm2_link_1_vhacd.obj scale=0.001 0.001 0.001; visual mesh filename=meshes/visual/arm2_link_1.obj scale=0.001 0.001 0.001
- link arm3_link_1: geometry collision mesh filename=meshes/collision/arm3_link_1_vhacd.obj scale=0.001 0.001 0.001; visual mesh filename=meshes/visual/arm3_link_1.obj scale=0.001 0.001 0.001
- link arm4_link_1: geometry collision mesh filename=meshes/collision/arm4_link_1_vhacd.obj scale=0.001 0.001 0.001; visual mesh filename=meshes/visual/arm4_link_1.obj scale=0.001 0.001 0.001
- link base_link: geometry collision mesh filename=meshes/collision/base_link_vhacd.obj scale=0.001 0.001 0.001; visual mesh filename=meshes/visual/base_link.obj scale=0.001 0.001 0.001
- link clamp2_link_1: geometry collision mesh filename=meshes/collision/clamp2_link_1_vhacd.obj scale=0.001 0.001 0.001; visual mesh filename=meshes/visual/clamp2_link_1.obj scale=0.001 0.001 0.001
- link clamp_arm_link_1: geometry collision mesh filename=meshes/collision/clamp_arm_link_1_vhacd.obj scale=0.001 0.001 0.001; visual mesh filename=meshes/visual/clamp_arm_link_1.obj scale=0.001 0.001 0.001
